Commit message: feat: add pinocchio dynamics package and rviz visualization

File: src/asr_sdm_universe/robot/asr_sdm_description/urdf/underwater_snakerobot.urdf (robot description, URDF)
Before this commit: robot underwater_snakerobot_description, 6 links, 5 joints
Links:
- link base_link: geometry visual mesh filename=package://asr_sdm_description/meshes/body_2links_head-blend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
- link link_2: geometry visual mesh filename=package://asr_sdm_description/meshes/body_2links.dae
- link screw_1_left: geometry visual mesh filename=package://asr_sdm_description/meshes/screw_left_CFD-blender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
- link screw_1_right: geometry visual mesh filename=package://asr_sdm_description/meshes/screw_right_CFD.dae
- link screw_2_left: geometry visual mesh filename=package://asr_sdm_description/meshes/screw_left_CFD.dae
- link screw_2_right: geometry visual mesh filename=package://asr_sdm_description/meshes/screw_right_CFD.dae
Joints:
- joint base_link_to_screw_1_left_joint: limit lower=-inf upper=inf effort=1000.0 velocity=10.0 -> lower=-3.14159 upper=3.14159 effort=1000.0 velocity=10.0
- joint base_link_to_screw_1_right_joint: limit lower=-inf upper=inf effort=1000.0 velocity=10.0 -> lower=-3.14159 upper=3.14159 effort=1000.0 velocity=10.0
- joint link_2_to_screw_2_left_joint: limit lower=-inf upper=inf effort=1000.0 velocity=10.0 -> lower=-3.14159 upper=3.14159 effort=1000.0 velocity=10.0
- joint link_2_to_screw_2_right_joint: limit lower=-inf upper=inf effort=1000.0 velocity=10.0 -> lower=-3.14159 upper=3.14159 effort=1000.0 velocity=10.0

File: src/asr_sdm_universe/robot/asr_sdm_description/urdf/underwater_snakerobot.urdf.xacro (robot description, xacro)
@@ -1,8 +1,12 @@
 <?xml version="1.0"?>
+<!--
+  Base xacro for the Amphibious Snake-like Robot.
+  Converted from the legacy package to use package:// URLs so meshes load
+  correctly from install space in ROS 2.
+-->
 <robot xmlns:xacro="http://www.ros.org/wiki/xacro" name="underwater_snakerobot_description">
 <!--................................. Definition ...................................-->
   <xacro:property name="pi" value="3.141592654" />
-  <xacro:property name="ext" value="osg" />
-  <xacro:property name="robot_parts_path" value="$(find underwater_snakerobot_description)/meshes" />
+  <xacro:property name="robot_parts_path" value="package://asr_sdm_description/meshes" />
 <!---............................. Link Definitions ................................-->
   <link name="base_link">
@@ -14,5 +18,5 @@
       <origin rpy="${pi} 0 ${-pi/2}" xyz="0.0 0.0 0.0"/>
       <geometry>
-        <mesh filename="${robot_parts_path}/body_2links_head-blender.${ext}"/>
+        <mesh filename="${robot_parts_path}/body_2links_head-blender.obj"/>
       </geometry>
     </visual>
@@ -22,5 +26,5 @@
       <origin rpy="${-pi} 0 ${pi/2}" xyz="0.0 0.0 0.0"/>
       <geometry>
-        <mesh filename="${robot_parts_path}/screw_left_CFD-blender.${ext}"/>
+        <mesh filename="${robot_parts_path}/screw_left_CFD-blender.obj"/>
       </geometry>
     </visual>
@@ -30,5 +34,5 @@
       <origin rpy="0 ${pi/2*3} 0" xyz="-0.0 0.0 0.0"/>
       <geometry>
-        <mesh filename="${robot_parts_path}/screw_right_CFD.${ext}"/>
+        <mesh filename="${robot_parts_path}/screw_right_CFD.dae"/>
       </geometry>
     </visual>
@@ -42,5 +46,5 @@
       <origin rpy="0 0 0" xyz="0.0 0.0 0.0"/>
       <geometry>
-        <mesh filename="${robot_parts_path}/body_2links.${ext}"/>
+        <mesh filename="${robot_parts_path}/body_2links.dae"/>
       </geometry>
     </visual>
@@ -50,5 +54,5 @@
       <origin rpy="0 ${pi/2*3} 0" xyz="0.0 0.0 0.0"/>
       <geometry>
-        <mesh filename="${robot_parts_path}/screw_left_CFD.${ext}"/>
+        <mesh filename="${robot_parts_path}/screw_left_CFD.dae"/>
       </geometry>
     </visual>
@@ -58,5 +62,5 @@
       <origin rpy="0 ${-pi/2} 0" xyz="-0.0 0.0 0.0"/>
       <geometry>
-        <mesh filename="${robot_parts_path}/screw_right_CFD.${ext}"/>
+        <mesh filename="${robot_parts_path}/screw_right_CFD.dae"/>
       </geometry>
     </visual>
@@ -67,5 +71,5 @@
     <child link="screw_1_left"/>
     <origin rpy="0 ${pi} 0" xyz="0.181 0 0"/>
-    <limit effort="1000.0" lower="-inf" upper="inf" velocity="10.0"/>
+    <limit effort="1000.0" lower="-3.14159" upper="3.14159" velocity="10.0"/>
     <safety_controller k_velocity="10" k_position="5"/>
   </joint>
@@ -74,5 +78,5 @@
     <child link="screw_1_right"/>
     <origin rpy="0 0 0" xyz="0.117 0 0"/>
-    <limit effort="1000.0" lower="-inf" upper="inf" velocity="10.0"/>
+    <limit effort="1000.0" lower="-3.14159" upper="3.14159" velocity="10.0"/>
     <safety_controller k_velocity="10" k_position="5"/>
   </joint>
@@ -88,5 +92,5 @@
     <child link="screw_2_left"/>
     <origin rpy="0 ${pi/2*3} 0" xyz="0 0 0.117"/>
-    <limit effort="1000.0" lower="-inf" upper="inf" velocity="10.0"/>
+    <limit effort="1000.0" lower="-3.14159" upper="3.14159" velocity="10.0"/>
     <safety_controller k_velocity="5" k_position="5"/>
   </joint>
@@ -95,5 +99,5 @@
     <child link="screw_2_right"/>
     <origin rpy="0 ${pi/2} 0" xyz="0 0 0.181"/>
-    <limit effort="1000.0" lower="-inf" upper="inf" velocity="10.0"/>
+    <limit effort="1000.0" lower="-3.14159" upper="3.14159" velocity="10.0"/>
     <safety_controller k_velocity="5" k_position="5"/>
   </joint>
